Commit message: update loss to support cross EEF

File: Assets/panda_gripper/panda_gripper_glb.urdf (robot description, URDF)
Before this commit: robot panda_gripper, 4 links, 3 joints
Links:
- added link panda_leftfinger_tip
- added link panda_rightfinger_tip
Joints:
- added joint panda_leftfinger_tip_joint: type fixed, parent panda_leftfinger, child panda_leftfinger_tip, origin xyz=0 0.00758 0.04525 rpy=0 0 0
- added joint panda_rightfinger_tip_joint: type fixed, parent panda_rightfinger, child panda_rightfinger_tip, origin xyz=0 -0.00758 0.04525 rpy=0 0 0

File: Assets/xarm7_panda_gripper/xarm7_panda_gripper.urdf (robot description, URDF)
Before this commit: robot xarm7_panda_gripper, 12 links, 11 joints
Links:
- added link panda_leftfinger_tip
- added link panda_rightfinger_tip
Joints:
- added joint panda_leftfinger_tip_joint: type fixed, parent panda_leftfinger, child panda_leftfinger_tip, origin xyz=0 0.00758 0.04525 rpy=0 0 0
- added joint panda_rightfinger_tip_joint: type fixed, parent panda_rightfinger, child panda_rightfinger_tip, origin xyz=0 -0.00758 0.04525 rpy=0 0 0
